Commit message: updated urdf

File: src/pothole_detector/urdf/bot1.urdf (robot description, URDF)
Before this commit: robot myfirst, 3 links, 2 joints
Links:
- removed link body_bot
- added link chasis; visual mesh filename=package://pothole_detector/meshes/body/bot2.dae
Joints:
- joint final_bot: parent body_bot -> chasis
- joint movingbot: parent body_bot -> chasis

Commit message: Add wheel mass and interia

File: src/pothole_detector/urdf/bot1.urdf (robot description, URDF)
Before this commit: robot Virat, 5 links, 4 joints
Links:
- link camera_link: mass 1e-5 -> None
- link castor_wheel: mass None -> 3
- link chasis: mass None -> 15.0
- link leftwheel: mass None -> 5
- link rightwheel: mass None -> 5
Joints:
- joint castorwheel_chasis: limit lower=-1.57 upper=1.57 effort=1 velocity=2 -> lower=-1.57 upper=1.57 effort=1 velocity=100
- joint leftwheel_chasis: limit lower=-1.57 upper=1.57 effort=1 velocity=2 -> lower=-1.57 upper=1.57 effort=1 velocity=100
- joint rightwheel_chasis: limit lower=-1.57 upper=1.57 effort=1 velocity=2 -> lower=-1.57 upper=1.57 effort=1 velocity=100

Commit message: Camera position fixed

File: src/pothole_detector/urdf/bot1.urdf (robot description, URDF)
Before this commit: robot Virat, 5 links, 4 joints
Links:
- removed link camera_link
- added link camera, mass 0.02; collision box size=${camera_size} ${camera_size} ${camera_size}; visual box size=${camera_size} ${camera_size} ${camera_size}
Joints:
- joint camera_joint: axis 0 1 0 -> (none); child camera_link -> camera; origin xyz=0.73 0 1.18 rpy=0 0.45 0 -> xyz=${camera_origin_x} ${camera_origin_y} ${camera_origin_z} rpy=0 0.45 0

Commit message: Teleop and opencv done

File: src/pothole_detector/urdf/bot1.urdf (robot description, URDF)
Before this commit: robot Virat, 5 links, 4 joints
Links:
- link castor_wheel: mass 3 -> 5; geometry collision mesh filename=package://pothole_detector/meshes/wheels/castors1.dae; visual mesh filename=package://pothole_detector/meshes/wheels/castors1.dae
- link chasis: mass 15.0 -> 15; geometry collision mesh filename=package://pothole_detector/meshes/wheels/bot2.dae; visual mesh filename=package://pothole_detector/meshes/body/bot2.dae
- link leftwheel: mass 5 -> 1; geometry collision mesh filename=package://pothole_detector/meshes/wheels/tyre1.dae; visual mesh filename=package://pothole_detector/meshes/wheels/tyre1.dae
- link rightwheel: mass 5 -> 1; geometry collision mesh filename=package://pothole_detector/meshes/wheels/tyre1.dae; visual mesh filename=package://pothole_detector/meshes/wheels/tyre1.dae
Joints:
- joint castorwheel_chasis: axis 0 0 1 -> 0 1 0; limit lower=-1.57 upper=1.57 effort=1 velocity=100 -> effort=1 velocity=100; type revolute -> fixed
- joint leftwheel_chasis: axis 0 0 1 -> 0 1 0; limit lower=-1.57 upper=1.57 effort=1 velocity=100 -> effort=1 velocity=100; type revolute -> continuous
- joint rightwheel_chasis: axis 0 0 1 -> 0 1 0; limit lower=-1.57 upper=1.57 effort=1 velocity=100 -> effort=1 velocity=100; type revolute -> continuous
